File: LineSensor/LineBoard_pro/LineBoard_pro.kicad_pcb (KiCad board)
At the start: 2 copper layers, 14 parts, among them J1 to MAIN

Commit message: 配線終わり
Parts:
- added C2: 0.1u, Capacitor_SMD:C_0603_1608Metric, F.Cu at (28.9, 44.3)
- added IC1: NJL7502R, NJL7502R:NJL7502R, F.Cu at (34.1, 34.7)
- added IC2: NJL7502R, NJL7502R:NJL7502R, F.Cu at (38.5, 34.7)
- added IC3: NJL7502R, NJL7502R:NJL7502R, F.Cu at (42.9, 34.7)
- added IC4: NJL7502R, NJL7502R:NJL7502R, F.Cu at (47.3, 34.7)
- added U1: TMUX1204DGSR, TMUX1204DGSR:DGS0010A-IPC_A, F.Cu at (31.3, 40.9)
Connections:
- J1 pad 3: /Line_A1 -> /Line_OUT
- J1 pad 4: /Line_S1 -> /Line_A0
- J1 pad 5: /Line_S2 -> /Line_A1
