File: LineSensor/LineBoard_pro/LineBoard_pro.kicad_pcb (KiCad board)
At the start: 2 copper layers, 20 parts, among them IC1 NJL7502R, IC2 NJL7502R, IC3 NJL7502R, IC4 NJL7502R, J1 to MAIN, U1 TMUX1204DGSR

Commit message: 部品仮配置
Parts:
- D1, D2, D3, D4, IC1, IC2, IC3, IC4, R2, R4, R6, R8: moved to B.Cu
- moved R7 101.4 mm to (122.7, 35.0), turned to 90 degrees
- moved R8 99.1 mm to (120.4, 37.7)
- moved D4 97.3 mm to (122.7, 35.0), turned to 90 degrees
- moved R5 91.8 mm to (113.1, 35.0), turned to 90 degrees
- moved R6 89.5 mm to (110.9, 37.7)
- moved D3 87.7 mm to (113.1, 35.0), turned to 90 degrees
- moved C1 72.7 mm to (91.8, 38.8), turned to 180 degrees
- moved IC4 72.7 mm to (120.0, 35.0), turned to 180 degrees
- moved J1 71.9 mm to (96.0, 40.0)
- moved R3 71.1 mm to (92.1, 35.0), turned to 90 degrees
- moved C2 70.2 mm to (98.6, 35.9)
- moved U1 69.1 mm to (100.0, 33.4)
- moved R4 68.9 mm to (89.9, 37.7)
- moved IC3 67.6 mm to (110.5, 35.0), turned to 180 degrees
- moved D2 66.9 mm to (92.1, 35.0), turned to 90 degrees
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Other:
- board text added: "S0"
- board text added: "S1"
- board text added: "S2"
- board text added: "S3"
