File: LineSensor/LineBoard_pro/LineBoard_pro.kicad_sch (KiCad schematic)
At the start: 18 parts, among them IC1 NJL7502R, IC2 NJL7502R, IC3 NJL7502R, IC4 NJL7502R, J1 to MAIN

Commit message: 配線終わり
Parts:
- added C2: 0.1u, Capacitor_SMD:C_0603_1608Metric, symbol Device:C_Small
- added U1: TMUX1204DGSR, TMUX1204DGSR:DGS0010A-IPC_A, symbol TMUX1204DGSR:TMUX1204DGSR
- IC1, IC2, IC3, IC4: footprint KiCad:NJL7502R -> NJL7502R:NJL7502R
Connections:
- net Line_S2 is gone; now on net Line_A1: J1.5 (Pin_5)
- net +3V3: now also C2.1, U1.5 (EN), U1.6 (VDD)
- net GND: now also C2.2, U1.3 (GND)
- net Line_A1: now also U1.10 (A1); no longer J1.3 (Pin_3)
- net S0: now also U1.2 (S1)
- net S1: now also U1.9 (S2)
- net S2: now also U1.4 (S3)
- net S3: now also U1.7 (S4)
- net Line_S1 renamed Line_A0
- net Line_A0: now also U1.1 (A0)
- new net Line_OUT: J1.3 (Pin_3), U1.8 (D)
